File: team6_pcb.kicad_sch (KiCad schematic)
At the start: 26 parts, among them P10 MAB, P2 STEP/DIR, P3 MISC, P4 Conn_01x01, P5 Conn_01x01, P8 VCC_IO, P9 VM, Q1 SI4532CDY-T1-GE3, Q2 SI4532CDY-T1-GE3, Q3 SI4532CDY-T1-GE3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

Commit message: Update team6_pcb.kicad_sch
Parts:
- R1, R2: value WSR2R0500FEA -> ERJ-3EKF10R0V; footprint Resistor_SMD:R_Shunt_Vishay_WSR2_WSR3 -> Resistor_SMD:R_0603_1608Metric
Changed lines of the file:
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@@
 			)
 		)
-		(property "Value" "WSR2R0500FEA"
+		(property "Value" "ERJ-3EKF10R0V"
 			(at 144.78 119.38 0)
 			(effects
@@
 			)
 		)
-		(property "Footprint" "Resistor_SMD:R_Shunt_Vishay_WSR2_WSR3"
+		(property "Footprint" "Resistor_SMD:R_0603_1608Metric"
 			(at 151.13 218.11 0)
 			(effects
@@
 			)
 		)
-		(property "Value" "WSR2R0500FEA"
+		(property "Value" "ERJ-3EKF10R0V"
 			(at 143.51 110.49 0)
 			(effects
@@
 			)
 		)
-		(property "Footprint" "Resistor_SMD:R_Shunt_Vishay_WSR2_WSR3"
+		(property "Footprint" "Resistor_SMD:R_0603_1608Metric"
 			(at 148.59 210.49 0)
 			(effects
