File: team6_pcb/team6_pcb.kicad_pcb (KiCad board)
At the start: 4 copper layers, 26 parts, among them P10 MAB, P2 STEP/DIR, P3 MISC, P4 Conn_01x01, P5 Conn_01x01, P8 VCC_IO, P9 VM, Q1 SI4532CDY-T1-GE3, Q2 SI4532CDY-T1-GE3, Q3 SI4532CDY-T1-GE3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

Commit message: team6_final_sumbits
Adin Stamped
Parts:
- added P1: SPI, Connector_PinHeader_2.54mm:PinHeader_1x04_P2.54mm_Vertical, F.Cu at (106.5, 99.5)
- moved D1 13.4 mm to (106.8, 114.4)
- moved R3 13.4 mm to (109.8, 113.9)
- turned R4 to 180 degrees
Connections:
- IC1 pad 10: unconnected-(IC1-SDO-Pad10) -> SDO
- IC1 pad 11: unconnected-(IC1-SDI-Pad11) -> SDI
- IC1 pad 12: unconnected-(IC1-SCK-Pad12) -> SCK
- IC1 pad 14: unconnected-(IC1-~{CS}-Pad14) -> CSN
Routing:
- net SRB: track 81.5 -> 3.88 mm
- net SRA: track 50.6 -> 14.3 mm
- net SDO: track 0.00 -> 23.8 mm, vias 0 -> 3
- net SDI: track 0.00 -> 21.1 mm, vias 0 -> 4
- net SCK: track 0.00 -> 16.6 mm, vias 0 -> 2
- net VCC_IO: track 48.2 -> 62.0 mm
- net CSN: track 0.00 -> 13.6 mm, vias 0 -> 2
- net LB2: track 48.8 -> 58.5 mm
- net LB1: track 60.4 -> 63.2 mm
- net GND: track 3.87 -> 5.52 mm, vias 38 -> 35
- net LA1: track 41.3 -> 40.2 mm
- net B2: vias 6 -> 5
- added copper zone on F.Cu, net GND
- added copper zone on F.Cu, net SRA
- added copper zone on F.Cu, net SRB
Other:
- board outline added: 52.8 x 52 mm
